Commit message: Add origins and axises

File: yamax.urdf (robot description, URDF)
Before this commit: robot yamax, 14 links, 13 joints
Joints:
- joint ankle_left: axis (none) -> 0 0 1; origin (none) -> xyz=0 0 0 rpy=0 0 0
- joint ankle_right: axis (none) -> 0 0 1; origin (none) -> xyz=0 0 0 rpy=0 0 0
- joint backbone_1: axis (none) -> 0 0 1; origin (none) -> xyz=0 3 0 rpy=0 0 0
- joint backbone_2: axis (none) -> 0 0 1; origin (none) -> xyz=0 0 0 rpy=0 0 0
- joint elbow_left: axis (none) -> 0 1 0; origin (none) -> xyz=0 0 0 rpy=0 0 1.5708
- joint elbow_right: axis (none) -> 0 1 0; origin (none) -> xyz=0 0 0 rpy=0 0 -1.5708
- joint hip_joint_left: axis (none) -> 0 0 1; origin (none) -> xyz=4 -1 0 rpy=0 0 0
- joint hip_joint_right: axis (none) -> 0 0 1; origin (none) -> xyz=-4 -1 0 rpy=0 0 0
- joint knee_left: axis (none) -> 0 0 1; origin (none) -> xyz=0 0 0 rpy=0 0 0
- joint knee_right: axis (none) -> 0 0 1; origin (none) -> xyz=0 0 0 rpy=0 0 0
- joint neck: axis (none) -> 0 1 0; origin (none) -> xyz=0 10 -1 rpy=0 0 0
- joint shoulder_left: axis (none) -> 0 1 0; origin (none) -> xyz=4 9 -1 rpy=0 0 1.5708
- joint shoulder_right: axis (none) -> 0 1 0; origin (none) -> xyz=-4 9 -1 rpy=0 0 -1.5708

Commit message: Add visual and place head and arms correctly

File: yamax.urdf (robot description, URDF)
Before this commit: robot yamax, 14 links, 13 joints
Links:
- added link arm_left_virtual
- added link arm_right_virtual
- link arm_left_1: geometry visual box size=1 5 0.5
- link arm_left_2: geometry visual box size=1 3 0.5
- link arm_right_1: geometry visual box size=1 5 0.5
- link arm_right_2: geometry visual box size=1 3 0.5
- link body: geometry visual box size=8 10 5
- link foot_left: geometry visual box size=4 1 5
- link foot_right: geometry visual box size=4 1 5
- link head: geometry visual box size=2.5 2 2
- link hip: geometry visual box size=8 1 5
- link leg_left_1: geometry visual box size=3 4 4
- link leg_left_2: geometry visual box size=3 4 4
- link leg_right_1: geometry visual box size=3 4 4
- link leg_right_2: geometry visual box size=3 4 4
- link stomach: geometry visual box size=3 4 6
Joints:
- added joint shoulder_left_2: type continuous, parent arm_left_virtual, child arm_left_1, origin xyz=0 0 0 rpy=0 0 0, axis 1 0 0
- added joint shoulder_right_2: type continuous, parent arm_right_virtual, child arm_right_1, origin xyz=0 0 0 rpy=0 0 0, axis 1 0 0
- joint ankle_left: axis 0 0 1 -> 1 0 0
- joint ankle_right: axis 0 0 1 -> 1 0 0
- joint elbow_left: axis 0 1 0 -> 0 0 1; origin xyz=0 0 0 rpy=0 0 1.5708 -> xyz=1 -4 -1 rpy=0 -1.5708 0
- joint elbow_right: axis 0 1 0 -> 0 0 1; origin xyz=0 0 0 rpy=0 0 -1.5708 -> xyz=-1 -4 -1 rpy=0 -1.5708 0
- joint knee_left: axis 0 0 1 -> 1 0 0
- joint knee_right: axis 0 0 1 -> 1 0 0
- joint neck: origin xyz=0 10 -1 rpy=0 0 0 -> xyz=0 6.5 -1 rpy=0 0 0
- joint shoulder_left: axis 0 1 0 -> 1 0 0; child arm_left_1 -> arm_left_virtual; origin xyz=4 9 -1 rpy=0 0 1.5708 -> xyz=5 4 -1 rpy=0 0 0
- joint shoulder_right: axis 0 1 0 -> 1 0 0; child arm_right_1 -> arm_right_virtual; origin xyz=-4 9 -1 rpy=0 0 -1.5708 -> xyz=-5 4 -1 rpy=0 0 0

Commit message: Fix naming and axis of the shoulder

File: yamax.urdf (robot description, URDF)
Before this commit: robot yamax, 16 links, 15 joints
Joints:
- removed joint shoulder_left
- removed joint shoulder_left_2
- removed joint shoulder_right
- removed joint shoulder_right_2
- added joint shoulder_left_x: type continuous, parent body, child arm_left_virtual, origin xyz=5 4 -1 rpy=0 0 0, axis 1 0 0
- added joint shoulder_left_z: type continuous, parent arm_left_virtual, child arm_left_1, origin xyz=0 0 0 rpy=0 0 0, axis 0 0 1
- added joint shoulder_right_x: type continuous, parent body, child arm_right_virtual, origin xyz=-5 4 -1 rpy=0 0 0, axis 1 0 0
- added joint shoulder_right_z: type continuous, parent arm_right_virtual, child arm_right_1, origin xyz=0 0 0 rpy=0 0 0, axis 0 0 1

Commit message: Decrease the height of body

File: yamax.urdf (robot description, URDF)
Before this commit: robot yamax, 16 links, 15 joints
Links:
- link body: geometry visual box size=8 6 5
Joints:
- joint backbone_1: origin xyz=0 3 0 rpy=0 0 0 -> xyz=0 -1 0 rpy=0 0 0
- joint neck: origin xyz=0 6.5 -1 rpy=0 0 0 -> xyz=0 4.5 -1 rpy=0 0 0
- joint shoulder_left_x: origin xyz=5 4 -1 rpy=0 0 0 -> xyz=5 2 -1 rpy=0 0 0
- joint shoulder_right_x: origin xyz=-5 4 -1 rpy=0 0 0 -> xyz=-5 2 -1 rpy=0 0 0

Commit message: Correct around the stomach

File: yamax.urdf (robot description, URDF)
Before this commit: robot yamax, 16 links, 15 joints
Links:
- added link backbone_virtual
- link hip: geometry visual box size=9 1 5
- link stomach: geometry visual box size=3 6 6
Joints:
- removed joint backbone_2
- added joint backbone_2_x: type continuous, parent stomach, child backbone_virtual, origin xyz=0 -6 0 rpy=0 0 0, axis 1 0 0
- added joint backbone_2_z: type continuous, parent backbone_virtual, child hip, origin xyz=0 0 0 rpy=0 0 0, axis 0 0 1
- joint backbone_1: origin xyz=0 -1 0 rpy=0 0 0 -> xyz=0 0 0 rpy=0 0 0

Commit message: Correct Legs

File: yamax.urdf (robot description, URDF)
Before this commit: robot yamax, 17 links, 16 joints
Links:
- added link leg_left_1_virtual
- added link leg_left_2_virtual
- added link leg_right_1_virtual
- added link leg_right_2_virtual
Joints:
- removed joint ankle_left
- removed joint ankle_right
- removed joint knee_left
- removed joint knee_right
- added joint ankle_left_x: type continuous, parent leg_left_2, child leg_left_2_virtual, origin xyz=0 -4.5 0 rpy=0 0 0, axis 1 0 0
- added joint ankle_left_z: type continuous, parent leg_left_2_virtual, child foot_left, origin xyz=0 0 0 rpy=0 0 0, axis 0 0 1
- added joint ankle_right_x: type continuous, parent leg_right_2, child leg_right_2_virtual, origin xyz=0 -4.5 0 rpy=0 0 0, axis 1 0 0
- added joint ankle_right_z: type continuous, parent leg_right_2_virtual, child foot_right, origin xyz=0 0 0 rpy=0 0 0, axis 0 0 1
- added joint knee_left_x: type continuous, parent leg_left_1, child leg_left_1_virtual, origin xyz=0 -4.5 0 rpy=0 0 0, axis 1 0 0
- added joint knee_left_z: type continuous, parent leg_left_1_virtual, child leg_left_2, origin xyz=0 0 0 rpy=0 0 0, axis 0 0 1
- added joint knee_right_x: type continuous, parent leg_right_1, child leg_right_1_virtual, origin xyz=0 -4.5 0 rpy=0 0 0, axis 1 0 0
- added joint knee_right_z: type continuous, parent leg_right_1_virtual, child leg_right_2, origin xyz=0 0 0 rpy=0 0 0, axis 0 0 1
- joint hip_joint_left: origin xyz=4 -1 0 rpy=0 0 0 -> xyz=2.5 -3 0 rpy=0 0 0
- joint hip_joint_right: origin xyz=-4 -1 0 rpy=0 0 0 -> xyz=-2.5 -3 0 rpy=0 0 0

Commit message: Some adjustments

File: yamax.urdf (robot description, URDF)
Before this commit: robot yamax, 21 links, 20 joints
Links:
- link arm_left_1: geometry visual box size=1 6 0.5
- link arm_left_2: geometry visual box size=1 5 0.5
- link arm_right_1: geometry visual box size=1 6 0.5
- link arm_right_2: geometry visual box size=1 5 0.5
- link foot_left: geometry visual box size=4 1 7
- link foot_right: geometry visual box size=4 1 7
- link stomach: geometry visual box size=3 5 3
Joints:
- joint backbone_1: origin xyz=0 0 0 rpy=0 0 0 -> xyz=0 0 1.5 rpy=0 0 0
- joint backbone_2_x: origin xyz=0 -6 0 rpy=0 0 0 -> xyz=0 -5 0 rpy=0 0 0
- joint hip_joint_left: origin xyz=2.5 -3 0 rpy=0 0 0 -> xyz=2.5 -2.5 0 rpy=0 0 0
- joint hip_joint_right: origin xyz=-2.5 -3 0 rpy=0 0 0 -> xyz=-2.5 -2.5 0 rpy=0 0 0
- joint neck: origin xyz=0 4.5 -1 rpy=0 0 0 -> xyz=0 4.5 0.5 rpy=0 0 0
- joint shoulder_left_x: origin xyz=5 2 -1 rpy=0 0 0 -> xyz=5 2 1 rpy=0 0 0
- joint shoulder_right_x: origin xyz=-5 2 -1 rpy=0 0 0 -> xyz=-5 2 1 rpy=0 0 0

Commit message: Remove unnecessary backbone_2_z

File: yamax.urdf (robot description, URDF)
Before this commit: robot yamax, 21 links, 20 joints
Links:
- removed link backbone_virtual
Joints:
- removed joint backbone_2_x
- removed joint backbone_2_z
- added joint backbone_2: type continuous, parent stomach, child hip, origin xyz=0 -5 0 rpy=0 0 0, axis 1 0 0

Commit message: Add limits (I didn't care about 'effort' and 'velocity')

File: yamax.urdf (robot description, URDF)
Before this commit: robot yamax, 20 links, 19 joints
Joints:
- joint ankle_left_x: limit (none) -> lower=-1.5708 upper=1.5708 effort=10 velocity=10; type continuous -> revolute
- joint ankle_left_z: limit (none) -> lower=-1.5708 upper=1.5708 effort=10 velocity=10; type continuous -> revolute
- joint ankle_right_x: limit (none) -> lower=-1.5708 upper=1.5708 effort=10 velocity=10; type continuous -> revolute
- joint ankle_right_z: limit (none) -> lower=-1.5708 upper=1.5708 effort=10 velocity=10; type continuous -> revolute
- joint backbone_1: limit (none) -> lower=-1.5708 upper=1.5708 effort=10 velocity=10; type continuous -> revolute
- joint backbone_2: limit (none) -> lower=-1.5708 upper=1.5708 effort=10 velocity=10; type continuous -> revolute
- joint elbow_left: limit (none) -> lower=-1.5708 upper=1.5708 effort=10 velocity=10; type continuous -> revolute
- joint elbow_right: limit (none) -> lower=-1.5708 upper=1.5708 effort=10 velocity=10; type continuous -> revolute
- joint hip_joint_left: limit (none) -> lower=-1.5708 upper=1.5708 effort=10 velocity=10; type continuous -> revolute
- joint hip_joint_right: limit (none) -> lower=-1.5708 upper=1.5708 effort=10 velocity=10; type continuous -> revolute
- joint knee_left_x: limit (none) -> lower=-1.5708 upper=1.5708 effort=10 velocity=10; type continuous -> revolute
- joint knee_left_z: limit (none) -> lower=-1.5708 upper=1.5708 effort=10 velocity=10; type continuous -> revolute
- joint knee_right_x: limit (none) -> lower=-1.5708 upper=1.5708 effort=10 velocity=10; type continuous -> revolute
- joint knee_right_z: limit (none) -> lower=-1.5708 upper=1.5708 effort=10 velocity=10; type continuous -> revolute
- joint neck: limit (none) -> lower=-1.5708 upper=1.5708 effort=10 velocity=10; type continuous -> revolute
- joint shoulder_left_x: limit (none) -> lower=-1.5708 upper=1.5708 effort=10 velocity=10; type continuous -> revolute
- joint shoulder_left_z: limit (none) -> lower=-1.5708 upper=1.5708 effort=10 velocity=10; type continuous -> revolute
- joint shoulder_right_x: limit (none) -> lower=-1.5708 upper=1.5708 effort=10 velocity=10; type continuous -> revolute
- joint shoulder_right_z: limit (none) -> lower=-1.5708 upper=1.5708 effort=10 velocity=10; type continuous -> revolute

Commit message: Remove unnecessary knee_{right,left}_z

File: yamax.urdf (robot description, URDF)
Before this commit: robot yamax, 20 links, 19 joints
Links:
- removed link leg_left_1_virtual
- removed link leg_right_1_virtual
Joints:
- removed joint knee_left_x
- removed joint knee_left_z
- removed joint knee_right_x
- removed joint knee_right_z
- added joint knee_left: type revolute, parent leg_left_1, child leg_left_2, origin xyz=0 -4.5 0 rpy=0 0 0, axis 1 0 0, limit lower=-1.5708 upper=1.5708 effort=10 velocity=10
- added joint knee_right: type revolute, parent leg_right_1, child leg_right_2, origin xyz=0 -4.5 0 rpy=0 0 0, axis 1 0 0, limit lower=-1.5708 upper=1.5708 effort=10 velocity=10

Commit message: Add z axis to hip_{right, left}

File: yamax.urdf (robot description, URDF)
Before this commit: robot yamax, 18 links, 17 joints
Links:
- added link hip_left_virtual
- added link hip_right_virtual
Joints:
- removed joint hip_joint_left
- removed joint hip_joint_right
- added joint hip_joint_left_x: type revolute, parent hip, child hip_left_virtual, origin xyz=2.5 -2.5 0 rpy=0 0 0, axis 1 0 0, limit lower=-1.5708 upper=1.5708 effort=10 velocity=10
- added joint hip_joint_left_z: type revolute, parent hip_left_virtual, child leg_left_1, origin xyz=0 0 0 rpy=0 0 0, axis 0 0 1, limit lower=-1.5708 upper=1.5708 effort=10 velocity=10
- added joint hip_joint_right_x: type revolute, parent hip, child hip_right_virtual, origin xyz=-2.5 -2.5 0 rpy=0 0 0, axis 1 0 0, limit lower=-1.5708 upper=1.5708 effort=10 velocity=10
- added joint hip_joint_right_z: type revolute, parent hip_right_virtual, child leg_right_1, origin xyz=0 0 0 rpy=0 0 0, axis 0 0 1, limit lower=-1.5708 upper=1.5708 effort=10 velocity=10

Commit message: Add collisions

File: yamax.urdf (robot description, URDF)
Before this commit: robot yamax, 20 links, 19 joints
Links:
- link arm_left_1: geometry collision box size=1 6 0.5; visual box size=1 6 0.5
- link arm_left_2: geometry collision box size=1 5 0.5; visual box size=1 5 0.5
- link arm_right_1: geometry collision box size=1 6 0.5; visual box size=1 6 0.5
- link arm_right_2: geometry collision box size=1 5 0.5; visual box size=1 5 0.5
- link body: geometry collision box size=8 6 5; visual box size=8 6 5
- link foot_left: geometry collision box size=4 1 7; visual box size=4 1 7
- link foot_right: geometry collision box size=4 1 7; visual box size=4 1 7
- link head: geometry collision box size=2.5 2 2; visual box size=2.5 2 2
- link hip: geometry collision box size=9 1 5; visual box size=9 1 5
- link leg_left_1: geometry collision box size=3 4 4; visual box size=3 4 4
- link leg_left_2: geometry collision box size=3 4 4; visual box size=3 4 4
- link leg_right_1: geometry collision box size=3 4 4; visual box size=3 4 4
- link leg_right_2: geometry collision box size=3 4 4; visual box size=3 4 4
- link stomach: geometry collision box size=3 5 3; visual box size=3 5 3

Commit message: Fixed the leg structure

File: yamax.urdf (robot description, URDF)
Before this commit: robot yamax, 20 links, 19 joints
Links:
- removed link leg_left_2_virtual
- removed link leg_right_2_virtual
- added link leg_left_3; collision box size=3 3 4; visual box size=3 3 4
- added link leg_right_3; collision box size=3 3 4; visual box size=3 3 4
- link hip_left_virtual: geometry collision box size=3 3 4; visual box size=3 3 4
- link hip_right_virtual: geometry collision box size=3 3 4; visual box size=3 3 4
- link leg_left_1: geometry collision box size=3 2 4; visual box size=3 2 4
- link leg_left_2: geometry collision box size=3 1 4; visual box size=3 1 4
- link leg_right_1: geometry collision box size=3 2 4; visual box size=3 2 4
- link leg_right_2: geometry collision box size=3 1 4; visual box size=3 1 4
Joints:
- removed joint ankle_left_x
- removed joint ankle_left_z
- removed joint ankle_right_x
- removed joint ankle_right_z
- added joint ankle_1_left: type revolute, parent leg_left_2, child leg_left_3, origin xyz=0 -1.5 0 rpy=0 0 0, axis 1 0 0, limit lower=-1.5708 upper=1.5708 effort=10 velocity=10
- added joint ankle_1_right: type revolute, parent leg_right_2, child leg_right_3, origin xyz=0 -1.5 0 rpy=0 0 0, axis 1 0 0, limit lower=-1.5708 upper=1.5708 effort=10 velocity=10
- added joint ankle_2_left: type revolute, parent leg_left_3, child foot_left, origin xyz=0 -3.5 0 rpy=0 0 0, axis 0 0 1, limit lower=-1.5708 upper=1.5708 effort=10 velocity=10
- added joint ankle_2_right: type revolute, parent leg_right_3, child foot_right, origin xyz=0 -3.5 0 rpy=0 0 0, axis 0 0 1, limit lower=-1.5708 upper=1.5708 effort=10 velocity=10
- joint hip_joint_left_x: child hip_left_virtual -> leg_left_1; origin xyz=2.5 -2.5 0 rpy=0 0 0 -> xyz=0 -3.5 0 rpy=0 0 0; parent hip -> hip_left_virtual
- joint hip_joint_left_z: child leg_left_1 -> hip_left_virtual; origin xyz=0 0 0 rpy=0 0 0 -> xyz=2.5 -1.5 0 rpy=0 0 0; parent hip_left_virtual -> hip
- joint hip_joint_right_x: child hip_right_virtual -> leg_right_1; origin xyz=-2.5 -2.5 0 rpy=0 0 0 -> xyz=0 -3.5 0 rpy=0 0 0; parent hip -> hip_right_virtual
- joint hip_joint_right_z: child leg_right_1 -> hip_right_virtual; origin xyz=0 0 0 rpy=0 0 0 -> xyz=-2.5 -1.5 0 rpy=0 0 0; parent hip_right_virtual -> hip
- joint knee_left: origin xyz=0 -4.5 0 rpy=0 0 0 -> xyz=0 -0.5 0 rpy=0 0 0
- joint knee_right: origin xyz=0 -4.5 0 rpy=0 0 0 -> xyz=0 -0.5 0 rpy=0 0 0

Commit message: Rename :)

File: yamax.urdf (robot description, URDF)
Before this commit: robot yamax, 20 links, 19 joints
Links:
- removed link hip_left_virtual
- removed link hip_right_virtual
- added link hip_left; collision box size=3 3 4; visual box size=3 3 4
- added link hip_right; collision box size=3 3 4; visual box size=3 3 4
Joints:
- joint hip_joint_left_x: parent hip_left_virtual -> hip_left
- joint hip_joint_left_z: child hip_left_virtual -> hip_left
- joint hip_joint_right_x: parent hip_right_virtual -> hip_right
- joint hip_joint_right_z: child hip_right_virtual -> hip_right

Commit message: Add xml verison tag and replace 'body' with 'base_link' to make it work propery

File: yamax.urdf (robot description, URDF)
Before this commit: robot yamax, 20 links, 19 joints
Links:
- removed link body
- added link base_link; collision box size=8 6 5; visual box size=8 6 5
Joints:
- joint backbone_1: parent body -> base_link
- joint neck: parent body -> base_link
- joint shoulder_left_x: parent body -> base_link
- joint shoulder_right_x: parent body -> base_link

Commit message: Use measured origins and sizes

File: yamax.urdf (robot description, URDF)
Before this commit: robot yamax, 20 links, 19 joints
Links:
- link arm_left_1: geometry collision box size=0.02 0.09 0.005; visual box size=0.02 0.09 0.005
- link arm_left_2: geometry collision box size=0.02 0.06 0.005; visual box size=0.02 0.06 0.005
- link arm_right_1: geometry collision box size=0.02 0.09 0.005; visual box size=0.02 0.09 0.005
- link arm_right_2: geometry collision box size=0.02 0.06 0.005; visual box size=0.02 0.06 0.005
- link base_link: geometry collision box size=0.11 0.094 0.05; visual box size=0.11 0.094 0.05
- link foot_left: geometry collision box size=0.060 0.005 0.090; visual box size=0.060 0.005 0.090
- link foot_right: geometry collision box size=0.060 0.005 0.090; visual box size=0.060 0.005 0.090
- link head: geometry collision box size=0.035 0.023 0.035; visual box size=0.035 0.023 0.035
- link hip: geometry collision box size=0.11 0.005 0.05; visual box size=0.11 0.005 0.05
- link hip_left: geometry collision box size=0.045 0.045 0.055; visual box size=0.045 0.045 0.055
- link hip_right: geometry collision box size=0.045 0.045 0.055; visual box size=0.045 0.045 0.055
- link leg_left_1: geometry collision box size=0.045 0.023 0.045; visual box size=0.045 0.023 0.045
- link leg_left_2: geometry collision box size=0.060 0.035 0.022; visual box size=0.060 0.035 0.022
- link leg_left_3: geometry collision box size=0.045 0.042 0.055; visual box size=0.045 0.042 0.055
- link leg_right_1: geometry collision box size=0.045 0.023 0.045; visual box size=0.045 0.023 0.045
- link leg_right_2: geometry collision box size=0.060 0.035 0.022; visual box size=0.060 0.035 0.022
- link leg_right_3: geometry collision box size=0.045 0.042 0.055; visual box size=0.045 0.042 0.055
- link stomach: geometry collision box size=0.053 0.070 0.054; visual box size=0.053 0.070 0.054
Joints:
- joint ankle_1_left: origin xyz=0 -1.5 0 rpy=0 0 0 -> xyz=0 -0.020 0 rpy=0 0 0
- joint ankle_1_right: origin xyz=0 -1.5 0 rpy=0 0 0 -> xyz=0 -0.020 0 rpy=0 0 0
- joint ankle_2_left: origin xyz=0 -3.5 0 rpy=0 0 0 -> xyz=0 -0.055 0.01 rpy=0 0 0
- joint ankle_2_right: origin xyz=0 -3.5 0 rpy=0 0 0 -> xyz=0 -0.055 0.01 rpy=0 0 0
- joint backbone_1: origin xyz=0 0 1.5 rpy=0 0 0 -> xyz=0 -0.020 0.005 rpy=0 0 0
- joint backbone_2: origin xyz=0 -5 0 rpy=0 0 0 -> xyz=0 -0.065 0 rpy=0 0 0
- joint elbow_left: origin xyz=1 -4 -1 rpy=0 -1.5708 0 -> xyz=0.020 -0.080 -0.010 rpy=0 -1.5708 0
- joint elbow_right: origin xyz=-1 -4 -1 rpy=0 -1.5708 0 -> xyz=-0.020 -0.080 -0.010 rpy=0 -1.5708 0
- joint hip_joint_left_x: origin xyz=0 -3.5 0 rpy=0 0 0 -> xyz=0 -0.050 0.010 rpy=0 0 0
- joint hip_joint_left_z: origin xyz=2.5 -1.5 0 rpy=0 0 0 -> xyz=0.035 -0.017 0 rpy=0 0 0
- joint hip_joint_right_x: origin xyz=0 -3.5 0 rpy=0 0 0 -> xyz=0 -0.050 0.010 rpy=0 0 0
- joint hip_joint_right_z: origin xyz=-2.5 -1.5 0 rpy=0 0 0 -> xyz=-0.035 -0.017 0 rpy=0 0 0
- joint knee_left: origin xyz=0 -0.5 0 rpy=0 0 0 -> xyz=0 -0.010 -0.010 rpy=0 0 0
- joint knee_right: origin xyz=0 -0.5 0 rpy=0 0 0 -> xyz=0 -0.010 -0.010 rpy=0 0 0
- joint neck: origin xyz=0 4.5 0.5 rpy=0 0 0 -> xyz=0 0.070 -0.005 rpy=0 0 0
- joint shoulder_left_x: origin xyz=5 2 1 rpy=0 0 0 -> xyz=0.075 0.040 0.025 rpy=0 0 0
- joint shoulder_right_x: origin xyz=-5 2 1 rpy=0 0 0 -> xyz=-0.075 0.040 0.025 rpy=0 0 0

Commit message: Replace 0.005 with 0.004

File: yamax.urdf (robot description, URDF)
Before this commit: robot yamax, 20 links, 19 joints
Links:
- link arm_left_1: geometry collision box size=0.02 0.09 0.004; visual box size=0.02 0.09 0.004
- link arm_left_2: geometry collision box size=0.02 0.06 0.004; visual box size=0.02 0.06 0.004
- link arm_right_1: geometry collision box size=0.02 0.09 0.004; visual box size=0.02 0.09 0.004
- link arm_right_2: geometry collision box size=0.02 0.06 0.004; visual box size=0.02 0.06 0.004
- link foot_left: geometry collision box size=0.060 0.004 0.090; visual box size=0.060 0.004 0.090
- link foot_right: geometry collision box size=0.060 0.004 0.090; visual box size=0.060 0.004 0.090
- link hip: geometry collision box size=0.11 0.004 0.05; visual box size=0.11 0.004 0.05
Joints:
- joint backbone_1: origin xyz=0 -0.020 0.005 rpy=0 0 0 -> xyz=0 -0.020 0.004 rpy=0 0 0
- joint neck: origin xyz=0 0.070 -0.005 rpy=0 0 0 -> xyz=0 0.070 -0.004 rpy=0 0 0
