Commit message: Fix axises

File: yamax.urdf (robot description, URDF)
Before this commit: robot yamax, 20 links, 19 joints
Links:
- link arm_left_1: geometry collision box size=0.004 0.02 0.09; visual box size=0.004 0.02 0.09
- link arm_left_2: geometry collision box size=0.004 0.02 0.06; visual box size=0.004 0.02 0.06
- link arm_right_1: geometry collision box size=0.004 0.02 0.09; visual box size=0.004 0.02 0.09
- link arm_right_2: geometry collision box size=0.004 0.02 0.06; visual box size=0.004 0.02 0.06
- link base_link: geometry collision box size=0.05 0.11 0.094; visual box size=0.05 0.11 0.094
- link foot_left: geometry collision box size=0.090 0.060 0.004; visual box size=0.090 0.060 0.004
- link foot_right: geometry collision box size=0.090 0.060 0.004; visual box size=0.090 0.060 0.004
- link head: geometry collision box size=0.035 0.035 0.023; visual box size=0.035 0.035 0.023
- link hip: geometry collision box size=0.05 0.11 0.004; visual box size=0.05 0.11 0.004
- link hip_left: geometry collision box size=0.055 0.045 0.045; visual box size=0.055 0.045 0.045
- link hip_right: geometry collision box size=0.055 0.045 0.045; visual box size=0.055 0.045 0.045
- link leg_left_1: geometry collision box size=0.045 0.045 0.023; visual box size=0.045 0.045 0.023
- link leg_left_2: geometry collision box size=0.022 0.060 0.035; visual box size=0.022 0.060 0.035
- link leg_left_3: geometry collision box size=0.055 0.045 0.042; visual box size=0.055 0.045 0.042
- link leg_right_1: geometry collision box size=0.045 0.045 0.023; visual box size=0.045 0.045 0.023
- link leg_right_2: geometry collision box size=0.022 0.060 0.035; visual box size=0.022 0.060 0.035
- link leg_right_3: geometry collision box size=0.055 0.045 0.042; visual box size=0.055 0.045 0.042
- link stomach: geometry collision box size=0.054 0.053 0.070; visual box size=0.054 0.053 0.070
Joints:
- joint ankle_1_left: axis 1 0 0 -> 0 1 0; origin xyz=0 -0.020 0 rpy=0 0 0 -> xyz=0 0 -0.020 rpy=0 0 0
- joint ankle_1_right: axis 1 0 0 -> 0 1 0; origin xyz=0 -0.020 0 rpy=0 0 0 -> xyz=0 0 -0.020 rpy=0 0 0
- joint ankle_2_left: axis 0 0 1 -> 1 0 0; origin xyz=0 -0.055 0.01 rpy=0 0 0 -> xyz=0.01 0 -0.055 rpy=0 0 0
- joint ankle_2_right: axis 0 0 1 -> 1 0 0; origin xyz=0 -0.055 0.01 rpy=0 0 0 -> xyz=0.01 0 -0.055 rpy=0 0 0
- joint backbone_1: axis 0 0 1 -> 1 0 0; origin xyz=0 -0.020 0.004 rpy=0 0 0 -> xyz=0.004 0 -0.020 rpy=0 0 0
- joint backbone_2: axis 1 0 0 -> 0 1 0; origin xyz=0 -0.065 0 rpy=0 0 0 -> xyz=0 0 -0.065 rpy=0 0 0
- joint elbow_left: axis 0 0 1 -> 1 0 0; origin xyz=0.020 -0.080 -0.010 rpy=0 -1.5708 0 -> xyz=-0.010 0.020 -0.080 rpy=0 0 -1.5708
- joint elbow_right: axis 0 0 1 -> 1 0 0; origin xyz=-0.020 -0.080 -0.010 rpy=0 -1.5708 0 -> xyz=-0.010 -0.020 -0.080 rpy=0 0 -1.5708
- joint hip_joint_left_x: axis 1 0 0 -> 0 1 0; origin xyz=0 -0.050 0.010 rpy=0 0 0 -> xyz=0.010 0 -0.050 rpy=0 0 0
- joint hip_joint_left_z: axis 0 0 1 -> 1 0 0; origin xyz=0.035 -0.017 0 rpy=0 0 0 -> xyz=0 0.035 -0.017 rpy=0 0 0
- joint hip_joint_right_x: axis 1 0 0 -> 0 1 0; origin xyz=0 -0.050 0.010 rpy=0 0 0 -> xyz=0.010 0 -0.050 rpy=0 0 0
- joint hip_joint_right_z: axis 0 0 1 -> 1 0 0; origin xyz=-0.035 -0.017 0 rpy=0 0 0 -> xyz=0 -0.035 -0.017 rpy=0 0 0
- joint knee_left: axis 1 0 0 -> 0 1 0; origin xyz=0 -0.010 -0.010 rpy=0 0 0 -> xyz=-0.010 0 -0.010 rpy=0 0 0
- joint knee_right: axis 1 0 0 -> 0 1 0; origin xyz=0 -0.010 -0.010 rpy=0 0 0 -> xyz=-0.010 0 -0.010 rpy=0 0 0
- joint neck: axis 0 1 0 -> 0 0 1; origin xyz=0 0.070 -0.004 rpy=0 0 0 -> xyz=-0.004 0 0.070 rpy=0 0 0
- joint shoulder_left_x: axis 1 0 0 -> 0 1 0; origin xyz=0.075 0.040 0.025 rpy=0 0 0 -> xyz=0.025 0.075 0.040 rpy=0 0 0
- joint shoulder_left_z: axis 0 0 1 -> 1 0 0
- joint shoulder_right_x: axis 1 0 0 -> 0 1 0; origin xyz=-0.075 0.040 0.025 rpy=0 0 0 -> xyz=0.025 -0.075 0.040 rpy=0 0 0
- joint shoulder_right_z: axis 0 0 1 -> 1 0 0

Commit message: Add inertial properties

File: yamax.urdf (robot description, URDF)
Before this commit: robot yamax, 20 links, 19 joints
Links:
- link arm_left_1: mass None -> 0.00914
- link arm_left_2: mass None -> 0.00355
- link arm_right_1: mass None -> 0.00914
- link arm_right_2: mass None -> 0.00355
- link base_link: mass None -> 0.233
- link foot_left: mass None -> 0.0209
- link foot_right: mass None -> 0.0209
- link head: mass None -> 0.0120
- link hip: mass None -> 0.072
- link hip_left: mass None -> 0.131
- link hip_right: mass None -> 0.131
- link leg_left_1: mass None -> 0.0599
- link leg_left_2: mass None -> 0.0036
- link leg_left_3: mass None -> 0.131
- link leg_right_1: mass None -> 0.0599
- link leg_right_2: mass None -> 0.0036
- link leg_right_3: mass None -> 0.131
- link stomach: mass None -> 0.00972
